Commit message: Defined the URDF better.

File: src/arduinobot_description/urdf/arduinobot.urdf.xacro (robot description, xacro)
@@ -1,4 +1,7 @@
 <?xml version="1.0"?>
 <robot xmlns:xacro = 'https://www.ros.org/wiki/xacro' name = 'arduinobot'>
+    <xacro:property name = "Pi" value = "3.14159"/>
+    <xacro:property name = "effort" value = "30.0"/>
+    <xacro:property name = "velocity" value = "10.0"/>
     <link name = "world"/>
     <link name = "base_link">
@@ -22,7 +25,84 @@
         </visual>
     </link>
-    <joint name = "joint_1" type = "fixed">
+    <joint name = "joint_1" type = "revolute">
         <parent link = "world"/>
         <child link = "base_plate"/>
+        <axis xyz = "0 0 1"/>
+        <origin rpy = "0 0 0" xyz = "0 0 0.307"/>
+        <limit lower = "-${Pi/2}" upper = "${Pi/2}" effort = "${effort}" velocity = "${velocity}"/>
+    </joint>
+    <link name = "forward_drive_arm">
+        <visual>
+            <origin rpy = "0 -${Pi/2} ${Pi/2}" xyz = "0.19 0.06 -0.08"/>
+            <geometry>
+                <mesh filename = "file:///home/faraz/arduinobot_ws/src/arduinobot_description/meshes/forward_drive_arm.STL" scale = "0.01 0.01 0.01"/>
+            </geometry>
+        </visual>
+    </link>
+    <joint name = "joint_2" type = "revolute">
+        <parent link = "base_plate"></parent>
+        <child link = "forward_drive_arm"/>
+        <axis xyz = "1 0 0"/>
+        <origin rpy = "0 0 0" xyz = "-.02 0 0.35"></origin>
+        <limit lower = "-${Pi/2}" upper = "${Pi/2}" effort = "${effort}" velocity = "${velocity}"/>
+    </joint>
+    <link name = "horizontal_arm">
+        <visual>
+            <origin rpy = "${Pi/2} 0 ${Pi/2}" xyz = "-0.03 -0.4 -0.06"/>
+            <geometry>
+                <mesh filename = "file:///home/faraz/arduinobot_ws/src/arduinobot_description/meshes/horizontal_arm.STL" scale = "0.01 0.01 0.01"/>
+            </geometry>
+        </visual>
+    </link>
+    <joint name = "joint_3" type = "revolute">
+        <parent link = "forward_drive_arm"/>
+        <child link = "horizontal_arm"/>
+        <axis xyz = "1 0 0"/>
+        <origin rpy = "0 0 0" xyz = "0 0 0.8"/>
+        <limit lower = "-${Pi/2}" upper = "${Pi/2}" effort = "${effort}" velocity = "${velocity}"/>
+    </joint>
+    <link name = "claw_support">
+        <visual>
+            <origin rpy = "0 0 ${Pi/2}" xyz = "-0 -0.05 -0.15"/>
+            <geometry>
+                <mesh filename = "file:///home/faraz/arduinobot_ws/src/arduinobot_description/meshes/claw_support.STL" scale = "0.01 0.01 0.01"/>
+            </geometry>
+        </visual>
+    </link>
+    <joint name = "horizontal_arm_to_claw_support" type = "fixed">
+        <parent link = "horizontal_arm"/>
+        <child link = "claw_support"/>
+        <origin xyz = "0 0.82 0" rpy = "0 0 0"/>
+    </joint>
+    <link name = "gripper_right">
+        <visual>
+            <origin rpy = "0 0 -${Pi/2}" xyz = "-0.1 0.5 -0.1"/>
+            <geometry>
+                <mesh filename = "file:///home/faraz/arduinobot_ws/src/arduinobot_description/meshes/right_finger.STL" scale = "0.01 0.01 0.01"/>
+            </geometry>
+        </visual>
+    </link>
+    <link name = "gripper_left">
+        <visual>
+            <origin rpy = "0 0 -${Pi/2}" xyz = "-0.04 0.5 -0.1"/>
+            <geometry>
+                <mesh filename = "file:///home/faraz/arduinobot_ws/src/arduinobot_description/meshes/left_finger.STL" scale = "0.01 0.01 0.01"/>
+            </geometry>
+        </visual>
+    </link>
+    <joint name = "joint_4" type = "revolute">
+        <parent link = "claw_support"/>
+        <child link = "gripper_right"/>
+        <axis xyz = "0 0 1"/>
+        <origin rpy = "0 0 0" xyz = "-0.04 0.13 -0.1"/>
+        <limit lower = "-${Pi/2}" upper = "${Pi/2}" effort = "${effort}" velocity = "${velocity}"/>
+    </joint>
+    <joint name = "joint_5" type = "revolute">
+        <parent link = "claw_support"/>
+        <child link = "gripper_left"/>
+        <axis xyz = "0 0 1"/>
+        <origin rpy = "0 0 0" xyz = "-0.22 0.13 -0.1"/>
+        <mimic joint = "joint_4" multiplier = "-1"/>
+        <limit lower = "0.0" upper = "${Pi/2}" effort = "${effort}" velocity = "${velocity}"/>
     </joint>
 </robot>

Commit message: Created and implemented a launch file in the workspace.

File: src/arduinobot_description/urdf/arduinobot.urdf.xacro (robot description, xacro)
@@ -106,3 +106,16 @@
         <limit lower = "0.0" upper = "${Pi/2}" effort = "${effort}" velocity = "${velocity}"/>
     </joint>
+    <link name = "rgb_camera">
+        <visual>
+            <origin rpy="-1.57 0 -1.57" xyz="-0.1 0.125 0.15"/>
+            <geometry>
+                <mesh filename = "file:///home/faraz/arduinobot_ws/src/arduinobot_description/meshes/pi_camera.STL" scale = "0.01 0.01 0.01"/>
+            </geometry>
+        </visual>
+    </link>
+    <joint name = "rgb_camera_joint" type = "fixed">
+        <parent link = "base_link"/>
+        <child link = "rgb_camera"/>
+        <origin xyz = "0 0 0" rpy = "0 0 0"/>
+    </joint>
 </robot>

Commit message: Created a gazebo launch file to spawn the robot in gazebo sim

File: src/arduinobot_description/urdf/arduinobot.urdf.xacro (robot description, xacro)
@@ -4,6 +4,15 @@
     <xacro:property name = "effort" value = "30.0"/>
     <xacro:property name = "velocity" value = "10.0"/>
+    <xacro:macro name = "default_inertial" params = "mass">
+        <inertial>
+            <mass value = "${mass}"/>
+            <inertia ixx = "1.0" ixy = "0.0" ixz = "0.0"
+                     iyy = "1.0" iyz = "0.0"
+                    izz = "1.0"/>
+        </inertial>
+    </xacro:macro>
     <link name = "world"/>
     <link name = "base_link">
+        <xacro:default_inertial mass = "1.0"/>
         <visual>
             <origin rpy = "0 0 0" xyz = "-0.5 -0.5 0"/>
@@ -12,4 +21,10 @@
             </geometry>
         </visual>
+        <collision>
+            <origin rpy = "0 0 0" xyz = "-0.5 -0.5 0"/>
+            <geometry>
+                <mesh filename = "file:///home/faraz/arduinobot_ws/src/arduinobot_description/meshes/basement.STL" scale = "0.01 0.01 0.01"/>
+            </geometry>
+        </collision>
     </link>
     <joint name = "virtual_joint" type = "fixed">
@@ -18,4 +33,5 @@
     </joint>
     <link name = "base_plate">
+        <xacro:default_inertial mass = "0.1"/>
         <visual>
             <origin rpy = "0 0 0" xyz = "-0.39 -0.39 -0.56"/>
@@ -24,4 +40,10 @@
             </geometry>
         </visual>
+        <collision>
+            <origin rpy = "0 0 0" xyz = "-0.39 -0.39 -0.56"/>
+            <geometry>
+                <mesh filename = "file:///home/faraz/arduinobot_ws/src/arduinobot_description/meshes/base_plate.STL" scale = "0.01 0.01 0.01"/>
+            </geometry>
+        </collision>
     </link>
     <joint name = "joint_1" type = "revolute">
@@ -33,4 +55,5 @@
     </joint>
     <link name = "forward_drive_arm">
+        <xacro:default_inertial mass = "0.1"/>
         <visual>
             <origin rpy = "0 -${Pi/2} ${Pi/2}" xyz = "0.19 0.06 -0.08"/>
@@ -39,4 +62,10 @@
             </geometry>
         </visual>
+        <collision>
+            <origin rpy = "0 -${Pi/2} ${Pi/2}" xyz = "0.19 0.06 -0.08"/>
+            <geometry>
+                <mesh filename = "file:///home/faraz/arduinobot_ws/src/arduinobot_description/meshes/forward_drive_arm.STL" scale = "0.01 0.01 0.01"/>
+            </geometry>
+        </collision>
     </link>
     <joint name = "joint_2" type = "revolute">
@@ -48,4 +77,5 @@
     </joint>
     <link name = "horizontal_arm">
+        <xacro:default_inertial mass = "0.1"/>
         <visual>
             <origin rpy = "${Pi/2} 0 ${Pi/2}" xyz = "-0.03 -0.4 -0.06"/>
@@ -54,4 +84,10 @@
             </geometry>
         </visual>
+        <collision>
+            <origin rpy = "${Pi/2} 0 ${Pi/2}" xyz = "-0.03 -0.4 -0.06"/>
+            <geometry>
+                <mesh filename = "file:///home/faraz/arduinobot_ws/src/arduinobot_description/meshes/horizontal_arm.STL" scale = "0.01 0.01 0.01"/>
+            </geometry>
+        </collision>
     </link>
     <joint name = "joint_3" type = "revolute">
@@ -63,4 +99,5 @@
     </joint>
     <link name = "claw_support">
+        <xacro:default_inertial mass = "0.05"/>
         <visual>
             <origin rpy = "0 0 ${Pi/2}" xyz = "-0 -0.05 -0.15"/>
@@ -69,4 +106,10 @@
             </geometry>
         </visual>
+        <collision>
+            <origin rpy = "0 0 ${Pi/2}" xyz = "-0 -0.05 -0.15"/>
+            <geometry>
+                <mesh filename = "file:///home/faraz/arduinobot_ws/src/arduinobot_description/meshes/claw_support.STL" scale = "0.01 0.01 0.01"/>
+            </geometry>
+        </collision>
     </link>
     <joint name = "horizontal_arm_to_claw_support" type = "fixed">
@@ -76,4 +119,5 @@
     </joint>
     <link name = "gripper_right">
+        <xacro:default_inertial mass = "0.01"/>
         <visual>
             <origin rpy = "0 0 -${Pi/2}" xyz = "-0.1 0.5 -0.1"/>
@@ -82,6 +126,13 @@
             </geometry>
         </visual>
+        <collision>
+            <origin rpy = "0 0 -${Pi/2}" xyz = "-0.1 0.5 -0.1"/>
+            <geometry>
+                <mesh filename = "file:///home/faraz/arduinobot_ws/src/arduinobot_description/meshes/right_finger.STL" scale = "0.01 0.01 0.01"/>
+            </geometry>
+        </collision>
     </link>
     <link name = "gripper_left">
+        <xacro:default_inertial mass = "0.01"/>
         <visual>
             <origin rpy = "0 0 -${Pi/2}" xyz = "-0.04 0.5 -0.1"/>
@@ -90,4 +141,10 @@
             </geometry>
         </visual>
+        <collision>
+            <origin rpy = "0 0 -${Pi/2}" xyz = "-0.04 0.5 -0.1"/>
+            <geometry>
+                <mesh filename = "file:///home/faraz/arduinobot_ws/src/arduinobot_description/meshes/left_finger.STL" scale = "0.01 0.01 0.01"/>
+            </geometry>
+        </collision>
     </link>
     <joint name = "joint_4" type = "revolute">
